File: pcb/led-o-clock.kicad_sch (KiCad schematic)
At the start: 22 parts, among them J1 USB_C_Receptacle_USB2.0_16P, J4 Led ring, J5 TX/RX/GND, SW3 IO9_BOOT, SW4 RST, U1 AP7361C-33E, U2 ESP32-C3-WROOM-02

Commit message: feat(pcb): work on v3.2
Parts:
- removed C1, C10, C7, C8, C9: 47uF, Capacitor_SMD:C_1206_3216Metric, symbol Device:C
- removed J5: TX/RX/GND, Connector_PinHeader_2.54mm:PinHeader_1x03_P2.54mm_Vertical, symbol Connector:Conn_01x03_Socket
- added C11: 100uF, Capacitor_SMD:CP_Elec_6.3x5.4, symbol Device:C_Polarized
- added FB1: FerriteBead_Small, Inductor_SMD:L_0603_1608Metric, symbol Device:FerriteBead_Small
Connections:
- net GND: now also C11.2
- net VCC_5V: now also C11.1, FB1.2; no longer C4.2, U1.1 (VI)
- new net: C4.2, FB1.1, U1.1 (VI)
